File: I2C Sensor Board_V2/16x2_LCD.kicad_sch (KiCad schematic)
At the start: 15 parts, among them Q3 2N7002, U11 PCF8574, U12 RC1602A

Commit message: Add files via upload
Connections:
- net +5V: now also R39.2; no longer Q3.3 (D)
- net GND: now also Q3.2 (S); no longer U12.16 (K)
- net Backlight: now reaches R37.1, U11.7 (P3)
- net at R39.1: now also U12.15 (A/VEE); no longer Q3.2 (S)
- new net: Q3.3 (D), U12.16 (K)
Other:
- moved on the sheet: Q3, R37, R38, R39
