File: I2C Sensor Board_V2/I2C Sensor Board_V2.kicad_pcb (KiCad board)
At the start: 4 copper layers, 160 x 100 mm, 203 parts, among them IC1 MCP6006UT-E_OT, J2 Conn_01x04_MountingPin, J3 Barrel_Jack_Switch, J4 Conn_02x03_Odd_Even, J5 USB_B, J6 Conn_01x02_Pin, J7 Conn_01x04_MountingPin, Q1 2N7002, Q2 2N7002, Q3 2N7002, Q4 PMOS, SW1 SW_DIP_x01, SW2 SW_DIP_x08, U1 ATmega328P-A, U10 MCP7940N-xSN, U11 PCF8574, U12 RC1602A, U13 PCA9685PW, U14 MCP3422Axx-xSN, U2 AP62300TWU, U3 CH340G, U4 LM75B, U5 PCF8574, U6 MCP9808_MSOP, U7 PCF8574, U8 24LC256, U9 MCP4725xxx-xCH, Y1 16 MHz, Y3 Crystal, Y4 12 MHz

Commit message: Add files via upload
Parts:
- added D13: D_Schottky, Diode_SMD:D_SOD-123F, F.Cu at (54.8, -8.65)
- added D14: Gr, LED_SMD:LED_0805_2012Metric_Pad1.15x1.40mm_HandSolder, F.Cu at (61.6, -18.5)
- added R26: 10k, Resistor_SMD:R_0805_2012Metric_Pad1.20x1.40mm_HandSolder, F.Cu at (61.6, -15.5)
- added TP16: TestPoint, TestPoint:TestPoint_THTPad_D1.5mm_Drill0.7mm, F.Cu at (50.3, -18.2)
- added TP17: TestPoint, TestPoint:TestPoint_THTPad_D1.5mm_Drill0.7mm, F.Cu at (50.3, -14.7)
- added TP18: TestPoint, TestPoint:TestPoint_THTPad_D1.5mm_Drill0.7mm, F.Cu at (50.3, -11.1)
- added TP19: TestPoint, TestPoint:TestPoint_THTPad_D1.5mm_Drill0.7mm, F.Cu at (37.3, -20.0)
- added TP20: TestPoint, TestPoint:TestPoint_THTPad_D1.5mm_Drill0.7mm, F.Cu at (37.3, -16.4)
- added TP21: TestPoint, TestPoint:TestPoint_THTPad_D1.5mm_Drill0.7mm, F.Cu at (37.3, -12.9)
- Q4: value PMOS -> FDN340P; footprint Created:SOT95P237X112-3N -> Package_TO_SOT_SMD:SOT-23
- moved TP7 188.3 mm to (24.5, 93.5)
- moved TP8 184.4 mm to (35.5, 93.5)
- moved C21 175.7 mm to (22.5, 85.0)
- moved JP16 175.7 mm to (34.5, 86.0)
- moved LED1 175.7 mm to (30.0, 85.5)
- moved R35 175.7 mm to (28.0, 89.0)
- moved R36 175.7 mm to (32.0, 89.0)
- moved U9 175.7 mm to (22.5, 88.0)
- moved Q4 51.3 mm to (60.0, -8.11)
- moved J4 13.2 mm to (54.7, 21.5)
- moved TP4 1.44 mm to (41.5, 6.50)
- moved TP1 1.15 mm to (52.5, 6.50)
- moved C10 1.00 mm to (143.0, 44.0)
- moved C6 1.00 mm to (135.0, 14.0)
- moved D10 1.00 mm to (136.0, 34.0)
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Connections:
- net Net-(U11-P3) renamed /16x2 LCD/Backlight
- C7 pad 2: +5V -> Net-(U2-SW)
- Q3 pad 2: Net-(Q3-S) -> GND
- Q3 pad 3: +5V -> Net-(Q3-D)
- Q4 pad 1: /MCU/USB_VCC -> Net-(IC1-VOUT)
- Q4 pad 2: Net-(IC1-VOUT) -> +5V
- Q4 pad 3: +5V -> /MCU/USB_VCC
- R39 pad 1: Net-(Q3-S) -> Net-(U12-A/VEE)
- R39 pad 2: Net-(U12-A/VEE) -> +5V
- U1 pad 1: /MCU/D3 -> /MCU/INT
- U1 pad 12: unconnected-(U1-PB0-Pad12) -> /MCU/D8
- U1 pad 13: unconnected-(U1-PB1-Pad13) -> /MCU/D9
- U1 pad 14: unconnected-(U1-PB2-Pad14) -> /MCU/D10
- U12 pad 16: GND -> Net-(Q3-D)
- U13 pad 26: /MCU/SDA -> /MCU/SCL
- U13 pad 27: /MCU/SCL -> /MCU/SDA
- U2 pad 3: +12V -> Net-(D13-K)
- U2 pad 5: Net-(U2-EN) -> unconnected-(U2-EN-Pad5)
- U7 pad 13: unconnected-(U7-~{INT}-Pad13) -> /MCU/INT
Routing:
- net /MCU/SDA: track 459.3 -> 429.0 mm
- net /MCU/INT: track 0.00 -> 20.8 mm, vias 0 -> 1
- net /MCU/D3: track 20.8 -> 0.00 mm, vias 1 -> 0
- net /MCU/SCL: track 456.5 -> 446.0 mm
- net GND: track 182.8 -> 191.2 mm, vias 95 -> 94
- net /MCU/SCK: track 16.3 -> 8.57 mm
- net /MCU/RST: track 39.1 -> 46.3 mm
- net Net-(U9-VOUT): track 17.8 -> 11.8 mm
- net Net-(Q3-S): track 4.80 -> 0.00 mm
- net (no net): track 0.00 -> 4.80 mm
- net /LM75 + LED + Fan/Heat: track 92.1 -> 88.0 mm
- net +5V: track 114.4 -> 110.7 mm, vias 73 -> 72
- net /LM75 + LED + Fan/Fan: track 105.9 -> 102.8 mm
- net Net-(Q3-D): track 0.00 -> 2.59 mm, vias 0 -> 1
