File: I2C Sensor Board_V2/I2C Sensor Board_V2.kicad_sch (KiCad schematic)
At the start: 6 parts

Commit message: Add files via upload
Other:
- sheet MCU ports: added INT; removed none
- sheet Mode Select ports: added INT; removed none
- moved on the sheet: TP1, TP2
