File: I2C Sensor Board_V2/Mode_Select.kicad_sch (KiCad schematic)
At the start: 14 parts, among them SW2 SW_DIP_x08, U7 PCF8574

Commit message: Add files via upload
Connections:
- net INT: now reaches U7.13 (~{INT})
- no-connect marks 1 -> 0
