File: I2C Sensor Board_V2/RGB.kicad_sch (KiCad schematic)
At the start: 25 parts, among them U13 PCA9685PW

Commit message: Add files via upload
Parts:
- added TP15: TestPoint, Created:Testpoint_5019_HandSolder, symbol Connector:TestPoint
Connections:
- net GND: now also TP15.1
- net SCL: now also U13.26 (SCL); no longer U13.27 (SDA)
- net SDA: now also U13.27 (SDA); no longer U13.26 (SCL)
